File: programmer_board/programmer_board.kicad_pcb (KiCad board)
At the start: 2 copper layers, 99.1 x 86.4 mm, 24 parts, among them J1 8bit_thing_bus_connector, J2 greenpak_i2c, U1 Pico, U2 74AHCT573, U3 74AHCT573, U4 74AHCT573, U5 74LVC245, U6 SLG46826G

Commit message: Completely reworked Pico programmer v1 board - final version
Parts:
- added C10: 100n, Capacitor_SMD:C_0805_2012Metric_Pad1.18x1.45mm_HandSolder, F.Cu at (84.2, 51.2)
- added C9: 100n, Capacitor_SMD:C_0805_2012Metric_Pad1.18x1.45mm_HandSolder, F.Cu at (62.7, 52.2)
- added JP1: Jumper_3_Bridged12, Connector_PinHeader_2.54mm:PinHeader_1x03_P2.54mm_Vertical, F.Cu at (114.7, 37.2)
- added REF**: TestPoint_THTPad_1.5x1.5mm_Drill0.7mm, TestPoint:TestPoint_THTPad_1.5x1.5mm_Drill0.7mm, F.Cu at (48.8, 64.0)
- added U7: 74LVC245, Package_SO:TSSOP-20_4.4x6.5mm_P0.65mm, F.Cu at (67.3, 56.1)
- added U8: 74LVC245, Package_SO:TSSOP-20_4.4x6.5mm_P0.65mm, F.Cu at (86.9, 56.1)
- moved C3 22.0 mm to (51.7, 50.3)
- moved G*** 21.6 mm to (58.4, 101.6)
- moved J2 15.1 mm to (123.7, 50.1), turned to -90 degrees
- moved R2 13.5 mm to (123.7, 53.4), turned to 90 degrees
- moved U5 13.3 mm to (47.8, 58.1)
- moved C1 12.6 mm to (43.2, 56.1), turned to -90 degrees
- moved C2 10.2 mm to (71.1, 48.4)
- moved R1 10.0 mm to (121.2, 53.4), turned to 90 degrees
- moved C5 9.91 mm to (109.2, 49.8)
- moved U6 9.91 mm to (114.0, 53.1)
- moved C6 9.91 mm to (116.7, 58.0)
- moved U2 9.48 mm to (57.4, 54.0)
- moved C4 4.47 mm to (90.8, 48.4)
- moved U4 4.37 mm to (96.5, 52.1)
- moved U3 2.52 mm to (77.0, 52.1)
Connections:
- J1 pad 37: /AS -> /C1
- J1 pad 39: unconnected-(J1-~{RESET}-Pad39) -> /~{RESET}
- J1 pad 40: unconnected-(J1-~{IRQ}-Pad40) -> /~{IRQ}
- U1 pad 10: /D5_OUT -> /~{A_H_LATCH_OE}
- U1 pad 11: /D6_OUT -> /D0_OUT
- U1 pad 12: /D7_OUT -> /D1_OUT
- U1 pad 14: /P_CLK -> /D2_OUT
- U1 pad 15: /A_L_LATCH -> /D3_OUT
- U1 pad 16: /A_H_LATCH -> /D4_OUT
- U1 pad 17: /~{P_STBY} -> /D5_OUT
- U1 pad 19: /P_AS -> /D6_OUT
- U1 pad 20: /P_R/~{W} -> /D7_OUT
- U1 pad 21: /D_LATCH -> /~{D_LATCH_OE}
- U1 pad 22: /D0_IN -> /D_LATCH
- U1 pad 24: /D1_IN -> /~{D_BUF_OE}
- U1 pad 25: /D2_IN -> /~{A_L_BUF_OE}
- U1 pad 26: /D3_IN -> /A_L_LATCH
- U1 pad 27: /D4_IN -> /~{A_L_LATCH_OE}
- U1 pad 29: /D5_IN -> /~{A_H_BUF_OE}
- U1 pad 31: /D6_IN -> /~{P_STBY}
- U1 pad 32: /D7_IN -> unconnected-(U1-GPIO27_ADC1-Pad32)
- U1 pad 34: /~{A_L_OE} -> unconnected-(U1-GPIO28_ADC2-Pad34)
- U1 pad 4: /D0_OUT -> /~{P_IRQ}
- U1 pad 5: /D1_OUT -> /P_C1
- U1 pad 6: /D2_OUT -> /P_CLK
- U1 pad 7: /D3_OUT -> /P_R/~{W}
- U1 pad 9: /D4_OUT -> /A_H_LATCH
- U2 pad 1: /~{D_OE} -> /~{D_LATCH_OE}
- U3 pad 1: /~{A_L_OE} -> /~{A_L_LATCH_OE}
- U4 pad 1: /~{STBY} -> /~{A_H_LATCH_OE}
- U5 pad 19: GND -> /~{D_BUF_OE}
- U5 pad 2: /D0_IN -> /D0_OUT
- U5 pad 3: /D1_IN -> /D1_OUT
- U5 pad 4: /D2_IN -> /D2_OUT
- U5 pad 5: /D3_IN -> /D3_OUT
- U5 pad 6: /D4_IN -> /D4_OUT
- U5 pad 7: /D5_IN -> /D5_OUT
- U5 pad 8: /D6_IN -> /D6_OUT
- U5 pad 9: /D7_IN -> /D7_OUT
- U6 pad 1: /~{P_STBY} -> /P_R/~{W}
- U6 pad 14: /AS -> /EXTRA_PIN
- U6 pad 16: /~{D_OE} -> /~{IRQ}
- U6 pad 2: /P_CLK -> /~{P_STBY}
- U6 pad 3: /P_AS -> /P_CLK
- U6 pad 4: /P_R/~{W} -> /P_C1
- U6 pad 8: unconnected-(U6-IO8-Pad8) -> /~{P_IRQ}
Routing:
- net /~{A_L_LATCH_OE}: track 0.00 -> 143.5 mm, vias 0 -> 4
- net /~{A_L_BUF_OE}: track 0.00 -> 115.9 mm, vias 0 -> 4
- net /~{A_H_BUF_OE}: track 0.00 -> 87.9 mm
- net /A_L_LATCH: track 46.2 -> 125.9 mm, vias 0 -> 2
- net +3.3V: track 177.3 -> 244.9 mm, vias 1 -> 7
- net /~{D_LATCH_OE}: track 0.00 -> 60.0 mm
- net /~{D_BUF_OE}: track 0.00 -> 58.1 mm
- net /~{P_IRQ}: track 0.00 -> 57.9 mm, vias 0 -> 2
- net /~{A_H_LATCH_OE}: track 0.00 -> 55.0 mm
- net /~{A_L_OE}: track 52.4 -> 0.00 mm
- net /~{P_STBY}: track 19.4 -> 70.2 mm
- net /P_C1: track 0.00 -> 50.8 mm
- net /~{D_OE}: track 45.5 -> 0.00 mm, vias 2 -> 0
- net /D7_IN: track 38.7 -> 0.00 mm
- net /D6_IN: track 37.2 -> 0.00 mm
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Other:
- board text added: "C1"
- board text added: "~{RESET}"
