File: midi/hardware/midi_board.kicad_pcb (KiCad board)
At the start: 2 copper layers, 99.1 x 86.4 mm, 41 parts, among them J1 MIDI OUT, J2 MIDI IN, J3 8bit_thing_bus_connector, J4 greenpak_i2c, J5 greenpak_i2c, J6 Conn_01x03_Pin, U1 6N137, U2 TL16C2550PFB, U3 SLG46826G, U4 SLG46826G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

Commit message: Final v1 version of the MIDI/UART board
- Tightened the layout a bit
- Added jumpers to select whether the second MIDI port is OUT or THRU
- Moved jumpers for system RX/TX connection to a better place
- Added labels for everything on the silkscreen
Parts:
- added JP3: Out/Thru select, own_footprints:PinHeader_1x03_P2.54mm_2_options_jumper_reverse, F.Cu at (57.7, 66.7)
Connections:
- U2 pad 7: Net-(U2-TXA) -> Net-(JP3-B)
- U5 pad 2: Net-(U2-TXA) -> Net-(JP3-C)
Routing:
- net Net-(U2-TXA): track 19.2 -> 0.00 mm
- net Net-(JP3-B): track 0.00 -> 15.1 mm
- net Net-(JP3-C): track 0.00 -> 4.11 mm
Other:
- board text added: "MIDI OUT/TRHU"
- board text added: "OUT"
- board text added: "SYS_RX"
- board text added: "SYS_TX"
- board text added: "TRHU"
- board text added: "UART"
- board text removed: "MIDI OUT"
- board text removed: "To System"
