File: io_board/hardware/io_board.kicad_pcb (KiCad board)
At the start: 2 copper layers, 99.1 x 86.4 mm, 34 parts, among them J1 8bit_thing_bus_connector, J2 greenpak_i2c, J3 greenpak_i2c, J4 Mini-DIN-6, J5 greenpak_i2c, J6 Micro_SD_Card_Det1, U1 SLG46826G, U2 W65C22, U3 SLG46826G, U4 74AHCT595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

Commit message: Route more of the io board
Parts:
- added BT1: Battery_Cell, Battery:BatteryHolder_MPD_BC2003_1x2032, F.Cu at (42.2, 95.5)
- added C10: 6.2p, Capacitor_SMD:C_0805_2012Metric_Pad1.18x1.45mm_HandSolder, F.Cu at (37.0, 78.8)
- added C11: 0.1u, Capacitor_SMD:C_0805_2012Metric_Pad1.18x1.45mm_HandSolder, F.Cu at (43.2, 75.9)
- added C8: 0.1u, Capacitor_SMD:C_0805_2012Metric_Pad1.18x1.45mm_HandSolder, F.Cu at (31.0, 65.5)
- added C9: 6.2p, Capacitor_SMD:C_0805_2012Metric_Pad1.18x1.45mm_HandSolder, F.Cu at (31.2, 78.8)
- added D1: BAT54W, Package_TO_SOT_SMD:SOT-323_SC-70, F.Cu at (46.2, 79.0)
- added R10: 1k, Resistor_SMD:R_0805_2012Metric_Pad1.20x1.40mm_HandSolder, F.Cu at (46.2, 74.7)
- added U7: MCP7940N-xP, Package_DIP:DIP-8_W7.62mm, F.Cu at (32.8, 75.2)
- added Y1: 32.768kHz, Crystal:Crystal_C26-LF_D2.1mm_L6.5mm_Horizontal, F.Cu at (33.2, 77.5)
- moved J6 6.14 mm to (64.3, 102.9)
- moved R4 2.05 mm to (37.0, 64.2)
- moved R3 2.05 mm to (34.0, 64.2)
Routing:
- net Net-(BT1-+): track 0.00 -> 39.8 mm
- net GND: track 14.5 -> 23.3 mm, vias 13 -> 27
- net Net-(U7-VBAT): track 0.00 -> 8.43 mm
- net +3.3V: track 33.4 -> 39.5 mm, vias 2 -> 0
- net /I2C_SCL: track 4.65 -> 10.2 mm
- net Net-(U7-X1): track 0.00 -> 4.48 mm
- net Net-(U7-X2): track 0.00 -> 4.42 mm
- net /I2C_SDA: track 4.69 -> 8.98 mm
- net Net-(D1-K): track 0.00 -> 3.73 mm
- net +5V: track 357.8 -> 360.2 mm
- net /SD_DI: track 35.9 -> 38.1 mm
- net /SD_DO: track 49.8 -> 51.9 mm
- net /~{SD_CS}: track 35.2 -> 36.9 mm
- net /SD_CLK: track 45.1 -> 46.7 mm
- added copper zone on F.Cu, net GND
